File: display.sch (KiCad schematic (older format))
At the start: 122 parts, among them P1 CONN_02X14, P2 CONN_02X15, Q1 BC846, Q10 BC846, Q11 BC856, Q12 BC856, Q13 BC846, Q14 BC846, Q15 BC856, Q16 BC856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

Commit message: Finishing layout, generating gerbers.
Parts:
- Q1, Q10, Q11, Q12, Q13, Q14, Q15, Q16, Q17, Q18, Q19, Q2, Q20, Q21, Q22, Q23, Q24, Q25, Q26, Q27, Q28, Q29, Q3, Q30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: footprint TO_SOT_Packages_SMD:SOT-23 -> TO_SOT_Packages_SMD:SOT-23_Handsoldering
